File: single_pot.kicad_pcb (KiCad board)
At the start: 2 copper layers, 22 x 18 mm, 7 parts, among them J1 I/O connector

Commit message: Reduce solder mask expansion to 0.05mm to fix aperture-bridge DRC
Other:
- rule pad_to_mask_clearance: 0.2 -> 0.05
Changed lines of the file:
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@@
       (dielectric_constraints no)
     )
-    (pad_to_mask_clearance 0.2)
+    (pad_to_mask_clearance 0.05)
     (pcbplotparams
       (layerselection 0x00010f0_ffffffff)
